File: Spankulator-Panel/SpankulatorPanel.kicad_pcb (KiCad board)
At the start: 2 copper layers, 60.4 x 128.4 mm, 29 parts

Commit message: Release 1.0
Full package.
Other:
- board text added: "Adjust/Activate"
- board text added: "Greenface Labs {dblquote}The Spankulator{dblquote} v3.4"
- board text removed: "Adjust"
- board text removed: "Greenface Labs "The Spankulator" v3.3"
- board text removed: "Push To Trigger"
- board text removed: "v3.3"
Changed lines of the file:
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@@
   (gr_line (start 98.2 79) (end 98.2 64) (layer "Edge.Cuts") (width 0.05))
   (gr_line (start 55 168.4) (end 115.4 168.4) (layer "Edge.Cuts") (width 0.05))
-  (gr_text "Greenface Labs\n\"The Spankulator\"\nv3.3" (at 85.75 161.75) (layer "B.SilkS")
+  (gr_text "Greenface Labs\n{dblquote}The Spankulator{dblquote}\nv3.4" (at 85.75 161.75) (layer "B.SilkS")
     (effects (font (size 1.5 1.5) (thickness 0.25)) (justify mirror))
   )
@@
     (effects (font (size 1.5 1.5) (thickness 0.3)))
   )
-  (gr_text "Push To\nTrigger" (at 85 116.3) (layer "F.SilkS")
-    (effects (font (size 1.5 1.5) (thickness 0.3)))
-  )
   (gr_text "12 HP -- WiFi Enabled" (at 86 165.5) (layer "F.SilkS")
     (effects (font (size 1 1) (thickness 0.15)))
   )
-  (gr_text "Adjust" (at 85.025 100.675) (layer "F.SilkS")
+  (gr_text "Adjust/Activate" (at 85.025 99.675) (layer "F.SilkS")
     (effects (font (size 1.5 1.5) (thickness 0.3)))
   )
@@
   (gr_text "<" (at 89.6 86) (layer "F.SilkS")
     (effects (font (size 4 3) (thickness 0.3)))
-  )
-  (gr_text "v3.3" (at 111.506 166.37) (layer "F.SilkS")
-    (effects (font (size 1.5 1.5) (thickness 0.15)))
   )
   (gr_text ">" (at 97.9 86) (layer "F.SilkS")
@@
   (zone (net 1) (net_name "GND") (layer "F.Cu") (hatch edge 0.508)
     (connect_pads (clearance 0.508))
-    (min_thickness 0.254)
+    (min_thickness 0.254) (filled_areas_thickness no)
     (fill yes (thermal_gap 0.508) (thermal_bridge_width 0.508))
     (polygon
@@
   (zone (net 0) (net_name "") (layer "B.Cu") (hatch edge 0.508)
     (connect_pads (clearance 0.508))
-    (min_thickness 0.254)
+    (min_thickness 0.254) (filled_areas_thickness no)
     (fill yes (thermal_gap 0.508) (thermal_bridge_width 0.508))
     (polygon
