File: Spankulator-Panel/SpankulatorPanel.kicad_pcb (KiCad board)
At the start: 2 copper layers, 60.4 x 128.4 mm, 29 parts

Commit message: New panel, new board.
Parts:
- removed G*** (x2): LOGO, panel:face_logo
- removed G***: LOGO, panel:dial2
- added dial1: SYM_Hot_Large, panel:dial2, F.Cu at (65.0, 146.7)
- added face1: SYM_Hot_Large, panel:partial3, F.Cu at (101.7, 130.8)
Other:
- board text added: "Greenface Labs {dblquote}The Spankulator{dblquote}"
- board text added: "Trig"
- board text removed: "Greenface Labs {dblquote}The Spankulator{dblquote} v3.4"
- board text removed: "Triggered"
