File: Spankulator-Panel/SpankulatorPanel.kicad_sch (KiCad schematic)
At the start: 26 parts

Commit message: New panel, new board.
Parts:
- added dial1: SYM_Hot_Large, panel:dial2, symbol Graphic:SYM_Hot_Large
- added face1: SYM_Hot_Large, panel:partial3, symbol Graphic:SYM_Hot_Large
Changed lines of the file:
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@@
-    )
-  )
-  (symbol (lib_id "Graphic:Logo_Open_Hardware_Small") (at 184.15 125.73 0) (unit 1)
-    (in_bom yes) (on_board yes)
-    (property "Reference" "#LOGO1" (id 0) (at 184.15 118.745 0)
-      (effects (font (size 1.27 1.27)) hide)
-    )
-    (property "Value" "Logo_Open_Hardware_Small" (id 1) (at 184.15 131.445 0)
-      (effects (font (size 1.27 1.27)) hide)
-    )
-    (property "Footprint" "" (id 2) (at 184.15 125.73 0)
-      (effects (font (size 1.27 1.27)) hide)
-    )
-    (property "Datasheet" "~" (id 3) (at 184.15 125.73 0)
-      (effects (font (size 1.27 1.27)) hide)
     )
   )
@@
     )
   )
+  (symbol (lib_name "SYM_Hot_Large_1") (lib_id "Graphic:SYM_Hot_Large") (at 123.825 114.935 0) (unit 1)
+    (in_bom yes) (on_board yes) (fields_autoplaced)
+    (property "Reference" "face1" (id 0) (at 123.825 109.855 0))
+    (property "Value" "SYM_Hot_Large" (id 1) (at 123.825 121.285 0)
+      (effects (font (size 1.27 1.27)) hide)
+    )
+    (property "Footprint" "panel:partial3" (id 2) (at 123.825 120.015 0)
+      (effects (font (size 1.27 1.27)) hide)
+    )
+    (property "Datasheet" "~" (id 3) (at 124.587 120.015 0)
+      (effects (font (size 1.27 1.27)) hide)
+    )
+  )
+  (symbol (lib_id "Graphic:SYM_Hot_Large") (at 145.415 114.935 0) (unit 1)
+    (in_bom yes) (on_board yes) (fields_autoplaced)
+    (property "Reference" "dial1" (id 0) (at 145.415 109.855 0))
+    (property "Value" "SYM_Hot_Large" (id 1) (at 145.415 121.285 0)
+      (effects (font (size 1.27 1.27)) hide)
+    )
+    (property "Footprint" "panel:dial2" (id 2) (at 145.415 120.015 0)
+      (effects (font (size 1.27 1.27)) hide)
+    )
+    (property "Datasheet" "~" (id 3) (at 146.177 120.015 0)
+      (effects (font (size 1.27 1.27)) hide)
+    )
+  )
   (sheet_instances
     (path "/" (page "1"))
   )
   (symbol_instances
-    (path "/00000000-0000-0000-0000-00005e4c6ad5"
-      (reference "#LOGO1") (unit 1) (value "Logo_Open_Hardware_Small") (footprint "")
-    )
     (path "/00000000-0000-0000-0000-00005e4a82ad"
       (reference "#PWR01") (unit 1) (value "GND") (footprint "")
@@
       (reference "H32") (unit 1) (value "MountingHole") (footprint "MountingHole:MountingHole_3.7mm")
     )
+    (path "/d94cd8c2-dfc5-473e-bce6-15458b288985"
+      (reference "dial1") (unit 1) (value "SYM_Hot_Large") (footprint "panel:dial2")
+    )
+    (path "/77b3938e-de7a-486c-b4c5-8f018d16467c"
+      (reference "face1") (unit 1) (value "SYM_Hot_Large") (footprint "panel:partial3")
+    )
   )
