File: DuDad/DuDad2HP-Board/DuDad2HP.kicad_pcb (KiCad board)
At the start: 2 copper layers, 10 x 110 mm, 22 parts, among them J1 EXP, J2 USB_B_Micro, J3 USB_A, Q1 MMBT5401, Q2 MMBT5401, Q3 2N7000, Q4 MMBT5401, SW1 Reset

Commit message: Consolidates zip_gerbers.bat. Improves BOM files.
Parts:
- J1: footprint Connector_PinHeader_2.54mm:PinHeader_2x05_P2.54mm_Vertical -> Connector_PinHeader_2.54mm:PinHeader_2x05_P2.54mm_Vertical_SMD
- Q3: value 2N7000 -> 2N7002
- moved R5 6.37 mm to (56.3, 84.6), turned to 90 degrees
- moved J1 5.07 mm to (55.0, 93.6)
- moved Q2 2.30 mm to (55.4, 79.7), turned to 90 degrees
- moved Q3 0.64 mm to (52.8, 134.8), turned to 0 degrees
Connections:
- Q2 pad 1: +3V3 -> Net-(R5-Pad2)
- Q2 pad 2: Net-(Q2-Pad2) -> +3V3
- Q3 pad 1: GND -> Net-(Q3-Pad1)
- Q3 pad 2: Net-(Q3-Pad2) -> GND
- Q4 pad 1: Net-(J2-Pad1) -> Net-(Q4-Pad1)
- Q4 pad 2: Net-(Q4-Pad2) -> Net-(J2-Pad1)
- R5 pad 2: Net-(Q2-Pad2) -> Net-(R5-Pad2)
- R6 pad 2: Net-(Q3-Pad2) -> Net-(Q3-Pad1)
- R7 pad 1: Net-(Q3-Pad2) -> Net-(Q3-Pad1)
- R8 pad 1: Net-(Q4-Pad2) -> Net-(Q4-Pad1)
- R9 pad 2: Net-(Q4-Pad2) -> Net-(Q4-Pad1)
Routing:
- net Net-(Q4-Pad1): track 0.00 -> 8.36 mm
- net Net-(J1-Pad10): track 10.8 -> 2.77 mm
- net Net-(Q4-Pad2): track 6.91 -> 0.00 mm
- net Net-(Q3-Pad2): track 6.91 -> 0.00 mm
- net Net-(Q3-Pad1): track 0.00 -> 6.44 mm
- net Net-(J2-Pad1): track 25.1 -> 21.3 mm
- net Net-(D3-Pad2): track 10.1 -> 6.62 mm, vias 0 -> 1
- net Net-(R5-Pad2): track 0.00 -> 2.97 mm
- net +3V3: track 26.4 -> 29.2 mm, vias 1 -> 3
- net Net-(Q2-Pad2): track 2.76 -> 0.00 mm
- net Net-(J1-Pad7): track 20.4 -> 18.3 mm
- net +12V: track 42.6 -> 43.6 mm, vias 2 -> 4
- net Net-(J1-Pad1): track 40.4 -> 40.1 mm, vias 0 -> 1

Commit message: Ups resistor values to dim LEDs. Adds generate BOMs.
Parts:
- Q1, Q2, Q4: value MMBT5401 -> MMBT3906
- R1, R4: value 200 -> 620
- R2, R5, R8: value 43K -> 30K
Other:
- board text added: "1.1."
- board text added: "v1.1"
- board text removed: "1.0."
- board text removed: "v1.0"
