File: DuDad/DuDad2HP-Board/DuDad2HP.kicad_sch (KiCad schematic)
At the start: 22 parts, among them J1 EXP, J2 USB_B_Micro, J3 USB_A, Q1 MMBT5401, Q2 MMBT5401, Q3 2N7000, Q4 MMBT5401, SW1 Reset

Commit message: Consolidates zip_gerbers.bat. Improves BOM files.
Parts:
- removed Q2: MMBT5401, Package_TO_SOT_SMD:SOT-23, symbol Transistor_BJT:2N3906
- added Q2: MMBT5401, Package_TO_SOT_SMD:SOT-23, symbol Transistor_BJT:MMBT3906
- J1: footprint Connector_PinHeader_2.54mm:PinHeader_2x05_P2.54mm_Vertical -> Connector_PinHeader_2.54mm:PinHeader_2x05_P2.54mm_Vertical_SMD;   LCSC Part # C225520 -> C124391
- Q3: value 2N7000 -> 2N7002; symbol Transistor_FET:2N7000 -> Transistor_FET:2N7002;   LCSC Part # C232838 -> C8545
- Q4: symbol Transistor_BJT:2N3906 -> Transistor_BJT:MMBT3906
Connections:
- net +3V3: now also Q2.2 (E)
- net GND: now also Q3.2 (S); no longer Q3.1 (S)
- net at R5.2: now also Q2.1 (B)
- net at D3.2 (A): now also Q2.3 (C)
- net at J2.1 (VBUS), R8.2: now also Q4.2 (E); no longer Q4.1 (E)
- net at R8.1, R9.2: now also Q4.1 (B); no longer Q4.2 (B)
- net at R6.2, R7.1: now also Q3.1 (G); no longer Q3.2 (G)
Changed lines of the file:
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@@
     )
-  )
-  (symbol (lib_id "Transistor_BJT:2N3906") (at 63.5 63.5 180) (unit 1)
-    (in_bom yes) (on_board yes)
-    (property "Reference" "Q2" (id 0) (at 58.674 64.6684 0)
-      (effects (font (size 1.27 1.27)) (justify left))
-    )
-    (property "Value" "MMBT5401" (id 1) (at 58.674 62.357 0)
-      (effects (font (size 1.27 1.27)) (justify left))
-    )
-    (property "Footprint" "Package_TO_SOT_SMD:SOT-23" (id 2) (at 58.42 61.595 0)
-      (effects (font (size 1.27 1.27) italic) (justify left) hide)
-    )
-    (property "Datasheet" "https://www.onsemi.com/pub/Collateral/2N3906-D.PDF" (id 3) (at 63.5 63.5 0)
-      (effects (font (size 1.27 1.27)) (justify left) hide)
-    )
-    (property "Digi-Key Part" "" (id 4) (at 63.5 63.5 0)
-      (effects (font (size 1.27 1.27)) hide)
-    )
-    (property "  LCSC Part #" "C8326" (id 5) (at 63.5 63.5 0)
-      (effects (font (size 1.27 1.27)) hide)
-    )
-    (pin "1")
-    (pin "2")
-    (pin "3")
   )
   (symbol (lib_id "Device:R_Small_US") (at 72.39 63.5 270) (unit 1)
@@
     (property "Reference" "J1" (id 0) (at 57.15 45.72 0))
     (property "Value" "EXP" (id 1) (at 57.15 48.26 0))
-    (property "Footprint" "Connector_PinHeader_2.54mm:PinHeader_2x05_P2.54mm_Vertical" (id 2) (at 55.88 38.1 0)
+    (property "Footprint" "Connector_PinHeader_2.54mm:PinHeader_2x05_P2.54mm_Vertical_SMD" (id 2) (at 55.88 38.1 0)
       (effects (font (size 1.27 1.27)) hide)
     )
@@
       (effects (font (size 1.27 1.27)) hide)
     )
-    (property "  LCSC Part #" "C225520" (id 5) (at 55.88 38.1 0)
+    (property "  LCSC Part #" "C124391" (id 5) (at 55.88 38.1 0)
       (effects (font (size 1.27 1.27)) hide)
     )
@@
     (pin "1")
   )
-  (symbol (lib_id "Transistor_BJT:2N3906") (at 120.65 80.645 270) (unit 1)
+  (symbol (lib_id "Transistor_BJT:MMBT3906") (at 120.65 80.645 270) (unit 1)
     (in_bom yes) (on_board yes)
     (property "Reference" "Q4" (id 0) (at 123.19 78.74 90)
@@
     )
     (property "  LCSC Part #" "C8326" (id 5) (at 120.65 80.645 0)
-      (effects (font (size 1.27 1.27)) hide)
-    )
-    (pin "1")
-    (pin "2")
-    (pin "3")
-  )
-  (symbol (lib_id "Transistor_BJT:MMBT3906") (at 34.29 63.5 180) (unit 1)
-    (in_bom yes) (on_board yes) (fields_autoplaced)
-    (property "Reference" "Q1" (id 0) (at 29.4386 62.5915 0)
-      (effects (font (size 1.27 1.27)) (justify left))
-    )
-    (property "Value" "MMBT5401" (id 1) (at 29.4386 65.3666 0)
-      (effects (font (size 1.27 1.27)) (justify left))
-    )
-    (property "Footprint" "Package_TO_SOT_SMD:SOT-23" (id 2) (at 29.21 61.595 0)
-      (effects (font (size 1.27 1.27) italic) (justify left) hide)
-    )
-    (property "Datasheet" "https://www.onsemi.com/pub/Collateral/2N3906-D.PDF" (id 3) (at 34.29 63.5 0)
-      (effects (font (size 1.27 1.27)) (justify left) hide)
-    )
-    (property "  LCSC Part #" "C8326" (id 4) (at 34.29 63.5 0)
       (effects (font (size 1.27 1.27)) hide)
     )
@@
     (pin "1")
   )
+  (symbol (lib_id "Transistor_BJT:MMBT3906") (at 63.5 63.5 180) (unit 1)
+    (in_bom yes) (on_board yes)
+    (property "Reference" "Q2" (id 0) (at 58.42 61.595 0)
+      (effects (font (size 1.27 1.27)) (justify left))
+    )
+    (property "Value" "MMBT5401" (id 1) (at 59.055 64.135 0)
+      (effects (font (size 1.27 1.27)) (justify left))
+    )
+    (property "Footprint" "Package_TO_SOT_SMD:SOT-23" (id 2) (at 58.42 61.595 0)
+      (effects (font (size 1.27 1.27) italic) (justify left) hide)
+    )
+    (property "Datasheet" "https://www.onsemi.com/pub/Collateral/2N3906-D.PDF" (id 3) (at 63.5 63.5 0)
+      (effects (font (size 1.27 1.27)) (justify left) hide)
+    )
+    (property "Digi-Key Part" "" (id 4) (at 63.5 63.5 0)
+      (effects (font (size 1.27 1.27)) hide)
+    )
+    (property "  LCSC Part #" "C8326" (id 5) (at 63.5 63.5 0)
+      (effects (font (size 1.27 1.27)) hide)
+    )
+    (pin "1")
+    (pin "2")
+    (pin "3")
+  )
   (symbol (lib_id "Device:R_Small_US") (at 131.445 62.865 270) (mirror x) (unit 1)
     (in_bom yes) (on_board yes)
@@
     (pin "2")
   )
-  (symbol (lib_id "Transistor_FET:2N7000") (at 172.72 74.295 0) (mirror y) (unit 1)
+  (symbol (lib_id "Transistor_FET:2N7002") (at 172.72 74.295 0) (mirror y) (unit 1)
     (in_bom yes) (on_board yes) (fields_autoplaced)
     (property "Reference" "Q3" (id 0) (at 167.5131 73.3865 0)
       (effects (font (size 1.27 1.27)) (justify left))
     )
-    (property "Value" "2N7000" (id 1) (at 167.5131 76.1616 0)
+    (property "Value" "2N7002" (id 1) (at 167.5131 76.1616 0)
       (effects (font (size 1.27 1.27)) (justify left))
     )
@@
       (effects (font (size 1.27 1.27)) hide)
     )
-    (property "  LCSC Part #" "C232838" (id 5) (at 172.72 74.295 0)
+    (property "  LCSC Part #" "C8545" (id 5) (at 172.72 74.295 0)
       (effects (font (size 1.27 1.27)) hide)
     )
@@
     (pin "2")
   )
+  (symbol (lib_id "Transistor_BJT:MMBT3906") (at 34.29 63.5 180) (unit 1)
+    (in_bom yes) (on_board yes)
+    (property "Reference" "Q1" (id 0) (at 29.21 61.595 0)
+      (effects (font (size 1.27 1.27)) (justify left))
+    )
+    (property "Value" "MMBT5401" (id 1) (at 29.845 64.135 0)
+      (effects (font (size 1.27 1.27)) (justify left))
+    )
+    (property "Footprint" "Package_TO_SOT_SMD:SOT-23" (id 2) (at 29.21 61.595 0)
+      (effects (font (size 1.27 1.27) italic) (justify left) hide)
+    )
+    (property "Datasheet" "https://www.onsemi.com/pub/Collateral/2N3906-D.PDF" (id 3) (at 34.29 63.5 0)
+      (effects (font (size 1.27 1.27)) (justify left) hide)
+    )
+    (property "Digi-Key Part" "" (id 4) (at 34.29 63.5 0)
+      (effects (font (size 1.27 1.27)) hide)
+    )
+    (property "  LCSC Part #" "C8326" (id 5) (at 34.29 63.5 0)
+      (effects (font (size 1.27 1.27)) hide)
+    )
+    (pin "1")
+    (pin "2")
+    (pin "3")
+  )
   (sheet_instances
     (path "/" (page "1"))
@@
     )
     (path "/00000000-0000-0000-0000-000062835217"
-      (reference "J1") (unit 1) (value "EXP") (footprint "Connector_PinHeader_2.54mm:PinHeader_2x05_P2.54mm_Vertical")
+      (reference "J1") (unit 1) (value "EXP") (footprint "Connector_PinHeader_2.54mm:PinHeader_2x05_P2.54mm_Vertical_SMD")
     )
     (path "/00000000-0000-0000-0000-0000627fe20b"
@@
       (reference "J3") (unit 1) (value "USB_A") (footprint "sputterizer:USB_A_Amphenol_UE27AE54100_Vertical")
     )
-    (path "/3e35ec55-6e98-4581-9a29-9732a6489518"
+    (path "/efd46df6-7130-4652-9949-fc9c1a4f0ff8"
       (reference "Q1") (unit 1) (value "MMBT5401") (footprint "Package_TO_SOT_SMD:SOT-23")
     )
-    (path "/00000000-0000-0000-0000-000061f47861"
+    (path "/7146301d-2b52-476f-b7bb-4b2a0a7e1026"
       (reference "Q2") (unit 1) (value "MMBT5401") (footprint "Package_TO_SOT_SMD:SOT-23")
     )
     (path "/92e94261-a13c-475b-b01e-c511c8f7e9b0"
-      (reference "Q3") (unit 1) (value "2N7000") (footprint "Package_TO_SOT_SMD:SOT-23")
+      (reference "Q3") (unit 1) (value "2N7002") (footprint "Package_TO_SOT_SMD:SOT-23")
     )
     (path "/21f9fd69-9bb1-463a-96ef-e2ad5cdcaa6c"

Commit message: Ups resistor values to dim LEDs. Adds generate BOMs.
Parts:
- J1:   LCSC Part # C124391 -> (none); LCSC Part # (none) -> C178296
- J3:   LCSC Part # C718031 -> (none); Digi-Key Part (none) -> UE27AE54100-ND; LCSC Part # (none) -> C386737
- Q1, Q2, Q4: value MMBT5401 -> MMBT3906;   LCSC Part # C8326 -> (none); Digi-Key Part (none) -> MMBT3906LT1GOSCT-ND; LCSC Part # (none) -> C266589
- Q3:   LCSC Part # C8545 -> (none); Digi-Key Part (none) -> 2N7002LT1GOSCT-ND; LCSC Part # (none) -> C8545
- R1, R4: value 200 -> 620;   LCSC Part # C17540 -> (none); Digi-Key Part (none) -> RMCF0805FT620RCT-ND; LCSC Part # (none) -> C17782
- R2, R5, R8: value 43K -> 30K;   LCSC Part # C17695 -> (none); Digi-Key Part (none) -> RMCF0805FT30K0CT-ND; LCSC Part # (none) -> C17621
- R3:   LCSC Part # C17513 -> (none); Digi-Key Part (none) -> 311-1.00KCRCT-ND; LCSC Part # (none) -> C17513
- R6, R9:   LCSC Part # C17414 -> (none); Digi-Key Part (none) -> RMCF0805FT10K0CT-ND; LCSC Part # (none) -> C17414
- R7:   LCSC Part # C17621 -> (none); Digi-Key Part (none) -> RMCF0805FT30K0CT-ND; LCSC Part # (none) -> C17621
