File: Spankulator-Hardware/parts.kicad_sch (KiCad schematic)
At the start: 42 parts, among them J11 OLED Pins, J14 Eurorack Power Cable, M2 OLED

Commit message: Uses correct knob for CV Adj
Parts:
- KN2: DK-Alt 1722-1314-ND -> (none); Digi-Key Part 1722-1241-ND -> 1722-1314-ND
Changed lines of the file:
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@@
       (effects (font (size 1.27 1.27)) hide)
     )
-    (property "Digi-Key Part" "1722-1241-ND" (id 4) (at 76.2 146.05 0)
+    (property "Digi-Key Part" "1722-1314-ND" (id 4) (at 76.2 146.05 0)
       (effects (font (size 1.27 1.27)) hide)
     )
-    (property "DK-Alt" "1722-1314-ND" (id 5) (at 76.2 146.05 0)
-      (effects (font (size 1.27 1.27)) hide)
-    )
